Commit message: add z1 arm to robot dog

File: source/robot_lab/data/Robots/unitree/b2_description/urdf/b2_description_b2z1.urdf (robot description, URDF)
Before this commit: robot b2_description, 45 links, 44 joints
Joints:
- joint z1_mount_joint: origin xyz=0.24 0.0 0.11 rpy=0 0 0 -> xyz=0.0 0.0 0.0 rpy=0 0 0
